File: led_controller_slave/led_controller_slave.kicad_pcb (KiCad board)
At the start: 2 copper layers, 108.7 x 46.7 mm, 60 parts, among them J1 Conn_01x06, J10 Conn_01x03, J11 Conn_01x03, J2 Conn_01x06, J3 Conn_01x03, J4 Conn_01x03, J5 Conn_01x03, J6 Conn_01x03, J7 Conn_01x03, J8 Conn_01x03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

Commit message: POC - first stage of development
Parts:
- added MH1: MountingHole_2.7mm_M2.5, MountingHole:MountingHole_2.7mm_M2.5, F.Cu at (62.0, 33.8)
- added MH2: MountingHole_2.7mm_M2.5, MountingHole:MountingHole_2.7mm_M2.5, F.Cu at (62.0, 50.0)
- added MH3: MountingHole_2.7mm_M2.5, MountingHole:MountingHole_2.7mm_M2.5, F.Cu at (128.5, 33.8)
- added MH4: MountingHole_2.7mm_M2.5, MountingHole:MountingHole_2.7mm_M2.5, F.Cu at (128.5, 50.0)
- added R25: 470R, Resistor_SMD:R_0805_2012Metric_Pad1.20x1.40mm_HandSolder, F.Cu at (143.5, 57.7)
- added R26: 470R, Resistor_SMD:R_0805_2012Metric_Pad1.20x1.40mm_HandSolder, F.Cu at (137.2, 57.7)
- added R27: 470R, Resistor_SMD:R_0805_2012Metric_Pad1.20x1.40mm_HandSolder, F.Cu at (130.8, 57.7)
- added R28: 470R, Resistor_SMD:R_0805_2012Metric_Pad1.20x1.40mm_HandSolder, F.Cu at (124.5, 57.7)
- added R29: 470R, Resistor_SMD:R_0805_2012Metric_Pad1.20x1.40mm_HandSolder, F.Cu at (118.1, 57.7)
- added R30: 470R, Resistor_SMD:R_0805_2012Metric_Pad1.20x1.40mm_HandSolder, F.Cu at (111.8, 57.7)
- added R31: 470R, Resistor_SMD:R_0805_2012Metric_Pad1.20x1.40mm_HandSolder, F.Cu at (105.2, 57.7)
- added R32: 470R, Resistor_SMD:R_0805_2012Metric_Pad1.20x1.40mm_HandSolder, F.Cu at (98.6, 57.7)
- added R33: 470R, Resistor_SMD:R_0805_2012Metric_Pad1.20x1.40mm_HandSolder, F.Cu at (92.5, 57.7)
- added R34: 470R, Resistor_SMD:R_0805_2012Metric_Pad1.20x1.40mm_HandSolder, F.Cu at (86.1, 57.7)
- added R35: 470R, Resistor_SMD:R_0805_2012Metric_Pad1.20x1.40mm_HandSolder, F.Cu at (80.0, 57.7)
- added R36: 470R, Resistor_SMD:R_0805_2012Metric_Pad1.20x1.40mm_HandSolder, F.Cu at (73.2, 57.7)
- added R37: 470R, Resistor_SMD:R_0805_2012Metric_Pad1.20x1.40mm_HandSolder, F.Cu at (67.1, 57.7)
- added R38: 470R, Resistor_SMD:R_0805_2012Metric_Pad1.20x1.40mm_HandSolder, F.Cu at (60.7, 57.7)
- added R39: 470R, Resistor_SMD:R_0805_2012Metric_Pad1.20x1.40mm_HandSolder, F.Cu at (54.6, 57.7)
- added R40: 470R, Resistor_SMD:R_0805_2012Metric_Pad1.20x1.40mm_HandSolder, F.Cu at (48.0, 57.6)
- moved Q1 2.03 mm to (142.5, 61.7)
- moved Q10 2.03 mm to (85.1, 61.7)
- moved Q11 2.03 mm to (79.1, 61.7)
- moved Q12 2.03 mm to (72.4, 61.9)
- moved Q13 2.03 mm to (66.0, 61.7)
- moved Q14 2.03 mm to (59.7, 61.7)
- moved Q15 2.03 mm to (53.7, 61.7)
- moved Q16 2.03 mm to (47.0, 61.7)
- moved Q2 2.03 mm to (136.1, 61.7)
- moved Q3 2.03 mm to (129.8, 61.7)
- moved Q6 2.03 mm to (110.7, 61.7)
- moved Q7 2.03 mm to (104.4, 61.7)
- moved Q8 2.03 mm to (97.8, 61.9)
- moved Q9 2.03 mm to (91.4, 61.9)
- moved Q4 2.03 mm to (123.4, 61.6)
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Connections:
- Q1 pad 1: G0 -> Net-(Q1-Pad1)
- Q10 pad 1: G9 -> Net-(Q10-Pad1)
- Q11 pad 1: G10 -> Net-(Q11-Pad1)
- Q12 pad 1: G11 -> Net-(Q12-Pad1)
- Q13 pad 1: G12 -> Net-(Q13-Pad1)
- Q14 pad 1: G13 -> Net-(Q14-Pad1)
- Q15 pad 1: G14 -> Net-(Q15-Pad1)
- Q16 pad 1: G15 -> Net-(Q16-Pad1)
- Q2 pad 1: G1 -> Net-(Q2-Pad1)
- Q3 pad 1: G2 -> Net-(Q3-Pad1)
- Q4 pad 1: G3 -> Net-(Q4-Pad1)
- Q5 pad 1: G4 -> Net-(Q5-Pad1)
- Q6 pad 1: G5 -> Net-(Q6-Pad1)
- Q7 pad 1: G6 -> Net-(Q7-Pad1)
- Q8 pad 1: G7 -> Net-(Q8-Pad1)
- Q9 pad 1: G8 -> Net-(Q9-Pad1)
Routing:
- net GND: track 317.0 -> 343.8 mm
- net G0: track 65.3 -> 60.4 mm
- net VCC: track 137.9 -> 134.2 mm
- net G4: track 42.5 -> 39.1 mm
- net G5: track 36.2 -> 33.2 mm
- net G9: track 21.4 -> 18.6 mm
- net LED4: track 11.1 -> 8.55 mm
- net LED8: track 10.6 -> 8.12 mm
- net LED7: track 11.2 -> 8.71 mm
- net LED3: track 11.5 -> 9.01 mm
- net LED11: track 11.3 -> 8.78 mm
- net G7: track 23.3 -> 20.8 mm
- net LED2: track 10.8 -> 8.34 mm
- net LED14: track 10.7 -> 8.31 mm
- net LED10: track 10.8 -> 8.34 mm
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Other:
- board size 108.7 x 46.7 mm -> 108.7 x 47.7 mm
