File: led_controller_slave/led_controller_slave.sch (KiCad schematic (older format))
At the start: 60 parts, among them J1 Conn_01x06, J10 Conn_01x03, J11 Conn_01x03, J2 Conn_01x06, J3 Conn_01x03, J4 Conn_01x03, J5 Conn_01x03, J6 Conn_01x03, J7 Conn_01x03, J8 Conn_01x03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

Commit message: POC - first stage of development
Parts:
- added R25, R26, R27, R28, R29, R30, R31, R32, R33, R34, R35, R36, R37, R38, R39, R40: 470R, Resistor_SMD:R_0805_2012Metric_Pad1.20x1.40mm_HandSolder, symbol Device:R
Connections:
- net G0: now also R25.1; no longer Q1.1
- net G1: now also R26.1; no longer Q2.1
- net G10: now also R35.1; no longer Q11.1
- net G11: now also R36.1; no longer Q12.1
- net G12: now also R37.1; no longer Q13.1
- net G13: now also R38.1; no longer Q14.1
- net G14: now also R39.1; no longer Q15.1
- net G15: now also R40.1; no longer Q16.1
- net G2: now also R27.1; no longer Q3.1
- net G3: now also R28.1; no longer Q4.1
- net G4: now also R29.1; no longer Q5.1
- net G5: now also R30.1; no longer Q6.1
- net G6: now also R31.1; no longer Q7.1
- net G7: now also R32.1; no longer Q8.1
- net G8: now also R33.1; no longer Q9.1
- net G9: now also R34.1; no longer Q10.1
- new net: Q1.1, R25.2
- new net: Q2.1, R26.2
- new net: Q3.1, R27.2
- new net: Q5.1, R29.2
- new net: Q6.1, R30.2
- new net: Q7.1, R31.2
- new net: Q4.1, R28.2
- new net: Q8.1, R32.2
- new net: Q12.1, R36.2
- new net: Q11.1, R35.2
- new net: Q10.1, R34.2
- new net: Q16.1, R40.2
- new net: Q15.1, R39.2
- new net: Q14.1, R38.2
- new net: Q13.1, R37.2
- new net: Q9.1, R33.2
